Commit message: Initial update for humble

File: rusty_description/urdf/materials.xacro (robot description, xacro)
@@ -2,32 +2,5 @@
 <robot name="rusty" xmlns:xacro="http://www.ros.org/wiki/xacro" >
 <material name="silver">
-    <color rgba="0.700 0.700 0.700 1.000"/>
-  </material>
-  <material name="black">
-    <color rgba="0.0 0.0 0.0 1.0"/>
-  </material>
-  <material name="blue">
-    <color rgba="0.0 0.0 0.8 1.0"/>
-  </material>
-  <material name="green">
-    <color rgba="0.0 0.8 0.0 1.0"/>
-  </material>
-  <material name="grey">
-    <color rgba="0.2 0.2 0.2 1.0"/>
-  </material>
-  <material name="orange">
-    <color rgba="${255/255} ${108/255} ${10/255} 1.0"/>
-  </material>
-  <material name="brown">
-    <color rgba="${222/255} ${207/255} ${195/255} 1.0"/>
-  </material>
-  <material name="yellow">
-    <color rgba="${0/255} ${180/255} ${180/255} 1.0"/>
-  </material>
-  <material name="red">
-    <color rgba="0.8 0.0 0.0 1.0"/>
-  </material>
-  <material name="white">
-    <color rgba="1.0 1.0 1.0 1.0"/>
-  </material>
+  <color rgba="0.700 0.700 0.700 1.000"/>
+</material>
 </robot>

File: rusty_description/urdf/rusty.xacro (robot description, xacro)
@@ -4,21 +4,21 @@
 <xacro:include filename="$(find rusty_description)/urdf/rusty.trans" />
 <xacro:include filename="$(find rusty_description)/urdf/rusty.gazebo" />
-<link name="rusty_base">
-  <inertial>
-    <origin rpy="0 0 0" xyz="0.0002544970294304579 -2.7411733823236023e-17 0.08341254857000653"/>
+<link name="base_link">
+  <inertial>
+    <origin xyz="0.0002544970294304579 -2.7411733823236023e-17 0.08341254857000653" rpy="0 0 0"/>
     <mass value="14.333340375312384"/>
-    <inertia ixx="0.173307" ixy="0.0" ixz="-0.000171" iyy="0.373229" iyz="0.0" izz="0.490917"/>
-  </inertial>
-  <visual>
-    <origin rpy="0 0 0" xyz="0 0 0"/>
-    <geometry>
-      <mesh filename="package://rusty_description/meshes/base_link.stl" scale="0.001 0.001 0.001"/>
-    </geometry>
-    <material name="white"/>
-  </visual>
-  <collision>
-    <origin rpy="0 0 0" xyz="0 0 0"/>
-    <geometry>
-      <mesh filename="package://rusty_description/meshes/base_link.stl" scale="0.001 0.001 0.001"/>
+    <inertia ixx="0.173307" iyy="0.373229" izz="0.490917" ixy="0.0" iyz="0.0" ixz="-0.000171"/>
+  </inertial>
+  <visual>
+    <origin xyz="0 0 0" rpy="0 0 0"/>
+    <geometry>
+      <mesh filename="file://$(find rusty_description)/meshes/base_link.stl" scale="0.001 0.001 0.001"/>
+    </geometry>
+    <material name="silver"/>
+  </visual>
+  <collision>
+    <origin xyz="0 0 0" rpy="0 0 0"/>
+    <geometry>
+      <mesh filename="file://$(find rusty_description)/meshes/base_link.stl" scale="0.001 0.001 0.001"/>
     </geometry>
   </collision>
@@ -26,19 +26,19 @@
 <link name="RW2_1">
   <inertial>
-    <origin rpy="0 0 0" xyz="1.3877787807814457e-17 -0.012499999999999983 0.0"/>
+    <origin xyz="1.3877787807814457e-17 -0.012499999999999983 0.0" rpy="0 0 0"/>
     <mass value="0.18260507298990683"/>
-    <inertia ixx="0.000124" ixy="-0.0" ixz="0.0" iyy="0.000228" iyz="0.0" izz="0.000124"/>
-  </inertial>
-  <visual>
-    <origin rpy="0 0 0" xyz="0.095 0.16 -0.05"/>
-    <geometry>
-      <mesh filename="package://rusty_description/meshes/RW2_1.stl" scale="0.001 0.001 0.001"/>
-    </geometry>
-    <material name="black"/>
-  </visual>
-  <collision>
-    <origin rpy="0 0 0" xyz="0.095 0.16 -0.05"/>
-    <geometry>
-      <mesh filename="package://rusty_description/meshes/RW2_1.stl" scale="0.001 0.001 0.001"/>
+    <inertia ixx="0.000124" iyy="0.000228" izz="0.000124" ixy="-0.0" iyz="0.0" ixz="0.0"/>
+  </inertial>
+  <visual>
+    <origin xyz="0.095 0.16 -0.05" rpy="0 0 0"/>
+    <geometry>
+      <mesh filename="file://$(find rusty_description)/meshes/RW2_1.stl" scale="0.001 0.001 0.001"/>
+    </geometry>
+    <material name="silver"/>
+  </visual>
+  <collision>
+    <origin xyz="0.095 0.16 -0.05" rpy="0 0 0"/>
+    <geometry>
+      <mesh filename="file://$(find rusty_description)/meshes/RW2_1.stl" scale="0.001 0.001 0.001"/>
     </geometry>
   </collision>
@@ -46,19 +46,19 @@
 <link name="RW1_1">
   <inertial>
-    <origin rpy="0 0 0" xyz="-1.3877787807814457e-17 -0.012499999999999983 6.938893903907228e-18"/>
+    <origin xyz="-1.3877787807814457e-17 -0.012499999999999983 6.938893903907228e-18" rpy="0 0 0"/>
     <mass value="0.1826050729899068"/>
-    <inertia ixx="0.000124" ixy="-0.0" ixz="-0.0" iyy="0.000228" iyz="0.0" izz="0.000124"/>
-  </inertial>
-  <visual>
-    <origin rpy="0 0 0" xyz="-0.095 0.16 -0.05"/>
-    <geometry>
-      <mesh filename="package://rusty_description/meshes/RW1_1.stl" scale="0.001 0.001 0.001"/>
-    </geometry>
-    <material name="black"/>
-  </visual>
-  <collision>
-    <origin rpy="0 0 0" xyz="-0.095 0.16 -0.05"/>
-    <geometry>
-      <mesh filename="package://rusty_description/meshes/RW1_1.stl" scale="0.001 0.001 0.001"/>
+    <inertia ixx="0.000124" iyy="0.000228" izz="0.000124" ixy="-0.0" iyz="0.0" ixz="-0.0"/>
+  </inertial>
+  <visual>
+    <origin xyz="-0.095 0.16 -0.05" rpy="0 0 0"/>
+    <geometry>
+      <mesh filename="file://$(find rusty_description)/meshes/RW1_1.stl" scale="0.001 0.001 0.001"/>
+    </geometry>
+    <material name="silver"/>
+  </visual>
+  <collision>
+    <origin xyz="-0.095 0.16 -0.05" rpy="0 0 0"/>
+    <geometry>
+      <mesh filename="file://$(find rusty_description)/meshes/RW1_1.stl" scale="0.001 0.001 0.001"/>
     </geometry>
   </collision>
@@ -66,19 +66,19 @@
 <link name="LW2_1">
   <inertial>
-    <origin rpy="0 0 0" xyz="0.0 0.012499999999999928 0.0"/>
+    <origin xyz="0.0 0.012499999999999928 0.0" rpy="0 0 0"/>
     <mass value="0.18260507298990683"/>
-    <inertia ixx="0.000124" ixy="0.0" ixz="-0.0" iyy="0.000228" iyz="-0.0" izz="0.000124"/>
-  </inertial>
-  <visual>
-    <origin rpy="0 0 0" xyz="0.095 -0.16 -0.05"/>
-    <geometry>
-      <mesh filename="package://rusty_description/meshes/LW2_1.stl" scale="0.001 0.001 0.001"/>
-    </geometry>
-    <material name="black"/>
-  </visual>
-  <collision>
-    <origin rpy="0 0 0" xyz="0.095 -0.16 -0.05"/>
-    <geometry>
-      <mesh filename="package://rusty_description/meshes/LW2_1.stl" scale="0.001 0.001 0.001"/>
+    <inertia ixx="0.000124" iyy="0.000228" izz="0.000124" ixy="0.0" iyz="-0.0" ixz="-0.0"/>
+  </inertial>
+  <visual>
+    <origin xyz="0.095 -0.16 -0.05" rpy="0 0 0"/>
+    <geometry>
+      <mesh filename="file://$(find rusty_description)/meshes/LW2_1.stl" scale="0.001 0.001 0.001"/>
+    </geometry>
+    <material name="silver"/>
+  </visual>
+  <collision>
+    <origin xyz="0.095 -0.16 -0.05" rpy="0 0 0"/>
+    <geometry>
+      <mesh filename="file://$(find rusty_description)/meshes/LW2_1.stl" scale="0.001 0.001 0.001"/>
     </geometry>
   </collision>
@@ -86,19 +86,19 @@
 <link name="LW1_1">
   <inertial>
-    <origin rpy="0 0 0" xyz="2.7755575615628914e-17 0.012500000000000039 2.0816681711721685e-17"/>
+    <origin xyz="2.7755575615628914e-17 0.012500000000000039 2.0816681711721685e-17" rpy="0 0 0"/>
     <mass value="0.1826050729899069"/>
-    <inertia ixx="0.000124" ixy="0.0" ixz="0.0" iyy="0.000228" iyz="0.0" izz="0.000124"/>
-  </inertial>
-  <visual>
-    <origin rpy="0 0 0" xyz="-0.095 -0.16 -0.05"/>
-    <geometry>
-      <mesh filename="package://rusty_description/meshes/LW1_1.stl" scale="0.001 0.001 0.001"/>
-    </geometry>
-    <material name="black"/>
-  </visual>
-  <collision>
-    <origin rpy="0 0 0" xyz="-0.095 -0.16 -0.05"/>
-    <geometry>
-      <mesh filename="package://rusty_description/meshes/LW1_1.stl" scale="0.001 0.001 0.001"/>
+    <inertia ixx="0.000124" iyy="0.000228" izz="0.000124" ixy="0.0" iyz="0.0" ixz="0.0"/>
+  </inertial>
+  <visual>
+    <origin xyz="-0.095 -0.16 -0.05" rpy="0 0 0"/>
+    <geometry>
+      <mesh filename="file://$(find rusty_description)/meshes/LW1_1.stl" scale="0.001 0.001 0.001"/>
+    </geometry>
+    <material name="silver"/>
+  </visual>
+  <collision>
+    <origin xyz="-0.095 -0.16 -0.05" rpy="0 0 0"/>
+    <geometry>
+      <mesh filename="file://$(find rusty_description)/meshes/LW1_1.stl" scale="0.001 0.001 0.001"/>
     </geometry>
   </collision>
@@ -106,19 +106,19 @@
 <link name="Holder_1">
   <inertial>
-    <origin rpy="0 0 0" xyz="-4.445233212745621e-17 0.0 0.012500000000000011"/>
+    <origin xyz="-4.445233212745621e-17 0.0 0.012500000000000011" rpy="0 0 0"/>
     <mass value="25.69775961700859"/>
-    <inertia ixx="0.165882" ixy="0.0" ixz="-0.0" iyy="0.4688" iyz="0.0" izz="0.632005"/>
-  </inertial>
-  <visual>
-    <origin rpy="0 0 0" xyz="-0.0 -0.0 -0.15"/>
-    <geometry>
-      <mesh filename="package://rusty_description/meshes/Holder_1.stl" scale="0.001 0.001 0.001"/>
-    </geometry>
-    <material name="black"/>
-  </visual>
-  <collision>
-    <origin rpy="0 0 0" xyz="-0.0 -0.0 -0.15"/>
-    <geometry>
-      <mesh filename="package://rusty_description/meshes/Holder_1.stl" scale="0.001 0.001 0.001"/>
+    <inertia ixx="0.165882" iyy="0.4688" izz="0.632005" ixy="0.0" iyz="0.0" ixz="-0.0"/>
+  </inertial>
+  <visual>
+    <origin xyz="-0.0 -0.0 -0.15" rpy="0 0 0"/>
+    <geometry>
+      <mesh filename="file://$(find rusty_description)/meshes/Holder_1.stl" scale="0.001 0.001 0.001"/>
+    </geometry>
+    <material name="silver"/>
+  </visual>
+  <collision>
+    <origin xyz="-0.0 -0.0 -0.15" rpy="0 0 0"/>
+    <geometry>
+      <mesh filename="file://$(find rusty_description)/meshes/Holder_1.stl" scale="0.001 0.001 0.001"/>
     </geometry>
   </collision>
@@ -126,19 +126,19 @@
 <link name="Lidar_1">
   <inertial>
-    <origin rpy="0 0 0" xyz="0.007402159277225678 -0.00023091322011423596 0.0050000000000000044"/>
+    <origin xyz="0.007402159277225678 -0.00023091322011423596 0.0050000000000000044" rpy="0 0 0"/>
     <mass value="0.008257286244679606"/>
-    <inertia ixx="1e-06" ixy="-0.0" ixz="0.0" iyy="0.0" iyz="0.0" izz="1e-06"/>
-  </inertial>
-  <visual>
-    <origin rpy="0 0 0" xyz="-0.235 -0.0 -0.135"/>
-    <geometry>
-      <mesh filename="package://rusty_description/meshes/Lidar_1.stl" scale="0.001 0.001 0.001"/>
-    </geometry>
-    <material name="blue"/>
-  </visual>
-  <collision>
-    <origin rpy="0 0 0" xyz="-0.235 -0.0 -0.135"/>
-    <geometry>
-      <mesh filename="package://rusty_description/meshes/Lidar_1.stl" scale="0.001 0.001 0.001"/>
+    <inertia ixx="1e-06" iyy="0.0" izz="1e-06" ixy="-0.0" iyz="0.0" ixz="0.0"/>
+  </inertial>
+  <visual>
+    <origin xyz="-0.235 -0.0 -0.135" rpy="0 0 0"/>
+    <geometry>
+      <mesh filename="file://$(find rusty_description)/meshes/Lidar_1.stl" scale="0.001 0.001 0.001"/>
+    </geometry>
+    <material name="silver"/>
+  </visual>
+  <collision>
+    <origin xyz="-0.235 -0.0 -0.135" rpy="0 0 0"/>
+    <geometry>
+      <mesh filename="file://$(find rusty_description)/meshes/Lidar_1.stl" scale="0.001 0.001 0.001"/>
     </geometry>
   </collision>
@@ -146,59 +146,59 @@
 <link name="Camera_1">
   <inertial>
-    <origin rpy="0 0 0" xyz="0.015039497744837121 0.0750001326555918 -0.02024300342659574"/>
+    <origin xyz="0.015039497744837121 0.0750001326555918 -0.02024300342659574" rpy="0 0 0"/>
     <mass value="0.007791207915918992"/>
-    <inertia ixx="1e-06" ixy="-0.0" ixz="-0.0" iyy="0.0" iyz="0.0" izz="1e-06"/>
-  </inertial>
-  <visual>
-    <origin rpy="0 0 0" xyz="-0.222588 -0.012099 -0.15"/>
-    <geometry>
-      <mesh filename="package://rusty_description/meshes/Camera_1.stl" scale="0.001 0.001 0.001"/>
-    </geometry>
-    <material name="black"/>
-  </visual>
-  <collision>
-    <origin rpy="0 0 0" xyz="-0.222588 -0.012099 -0.15"/>
-    <geometry>
-      <mesh filename="package://rusty_description/meshes/Camera_1.stl" scale="0.001 0.001 0.001"/>
+    <inertia ixx="1e-06" iyy="0.0" izz="1e-06" ixy="-0.0" iyz="0.0" ixz="-0.0"/>
+  </inertial>
+  <visual>
+    <origin xyz="-0.222588 -0.012099 -0.15" rpy="0 0 0"/>
+    <geometry>
+      <mesh filename="file://$(find rusty_description)/meshes/Camera_1.stl" scale="0.001 0.001 0.001"/>
+    </geometry>
+    <material name="silver"/>
+  </visual>
+  <collision>
+    <origin xyz="-0.222588 -0.012099 -0.15" rpy="0 0 0"/>
+    <geometry>
+      <mesh filename="file://$(find rusty_description)/meshes/Camera_1.stl" scale="0.001 0.001 0.001"/>
     </geometry>
   </collision>
 </link>
 <joint name="RW2" type="continuous">
-  <origin rpy="0 0 0" xyz="-0.095 -0.16 0.05"/>
-  <parent link="rusty_base"/>
+  <origin xyz="-0.095 -0.16 0.05" rpy="0 0 0"/>
+  <parent link="base_link"/>
   <child link="RW2_1"/>
-  <axis xyz="0.0 1.0 0.0"/>
+  <axis xyz="0.0 -1.0 0.0"/>
 </joint>
 <joint name="RW1" type="continuous">
-  <origin rpy="0 0 0" xyz="0.095 -0.16 0.05"/>
-  <parent link="rusty_base"/>
+  <origin xyz="0.095 -0.16 0.05" rpy="0 0 0"/>
+  <parent link="base_link"/>
   <child link="RW1_1"/>
   <axis xyz="0.0 1.0 0.0"/>
 </joint>
 <joint name="LW2" type="continuous">
-  <origin rpy="0 0 0" xyz="-0.095 0.16 0.05"/>
-  <parent link="rusty_base"/>
+  <origin xyz="-0.095 0.16 0.05" rpy="0 0 0"/>
+  <parent link="base_link"/>
   <child link="LW2_1"/>
-  <axis xyz="0.0 1.0 0.0"/>
+  <axis xyz="0.0 -1.0 0.0"/>
 </joint>
 <joint name="LW1" type="continuous">
-  <origin rpy="0 0 0" xyz="0.095 0.16 0.05"/>
-  <parent link="rusty_base"/>
+  <origin xyz="0.095 0.16 0.05" rpy="0 0 0"/>
+  <parent link="base_link"/>
   <child link="LW1_1"/>
   <axis xyz="0.0 1.0 0.0"/>
 </joint>
-<joint name="Rigid10" type="fixed">
-  <origin rpy="0 0 0" xyz="0.0 0.0 0.15"/>
-  <parent link="rusty_base"/>
+<joint name="Rigid 10" type="fixed">
+  <origin xyz="0.0 0.0 0.15" rpy="0 0 0"/>
+  <parent link="base_link"/>
   <child link="Holder_1"/>
 </joint>
-<joint name="Rigid11" type="fixed">
-  <origin rpy="0 0 0" xyz="0.235 0.0 0.135"/>
-  <parent link="rusty_base"/>
+<joint name="Rigid 11" type="fixed">
+  <origin xyz="0.235 0.0 0.135" rpy="0 0 0"/>
+  <parent link="base_link"/>
   <child link="Lidar_1"/>
 </joint>
-<joint name="Rigid12" type="fixed">
-  <origin rpy="0 0 0" xyz="0.222588 0.012099 0.15"/>
-  <parent link="rusty_base"/>
+<joint name="Rigid 12" type="fixed">
+  <origin xyz="0.222588 0.012099 0.15" rpy="0 0 0"/>
+  <parent link="base_link"/>
   <child link="Camera_1"/>
 </joint>

Commit message: updated laser and cmd_vel plugin with visuals for the robot

File: rusty_description/urdf/materials.xacro (robot description, xacro)
@@ -2,5 +2,32 @@
 <robot name="rusty" xmlns:xacro="http://www.ros.org/wiki/xacro" >
 <material name="silver">
-  <color rgba="0.700 0.700 0.700 1.000"/>
-</material>
+    <color rgba="0.700 0.700 0.700 1.000"/>
+  </material>
+  <material name="black">
+    <color rgba="0.0 0.0 0.0 1.0"/>
+  </material>
+  <material name="blue">
+    <color rgba="0.0 0.0 0.8 1.0"/>
+  </material>
+  <material name="green">
+    <color rgba="0.0 0.8 0.0 1.0"/>
+  </material>
+  <material name="grey">
+    <color rgba="0.2 0.2 0.2 1.0"/>
+  </material>
+  <material name="orange">
+    <color rgba="${255/255} ${108/255} ${10/255} 1.0"/>
+  </material>
+  <material name="brown">
+    <color rgba="${222/255} ${207/255} ${195/255} 1.0"/>
+  </material>
+  <material name="yellow">
+    <color rgba="${0/255} ${180/255} ${180/255} 1.0"/>
+  </material>
+  <material name="red">
+    <color rgba="0.8 0.0 0.0 1.0"/>
+  </material>
+  <material name="white">
+    <color rgba="1.0 1.0 1.0 1.0"/>
+  </material>
 </robot>

File: rusty_description/urdf/rusty.xacro (robot description, xacro)
@@ -168,5 +168,5 @@
   <parent link="base_link"/>
   <child link="RW2_1"/>
-  <axis xyz="0.0 -1.0 0.0"/>
+  <axis xyz="0.0 1.0 0.0"/>
 </joint>
 <joint name="RW1" type="continuous">
@@ -180,5 +180,5 @@
   <parent link="base_link"/>
   <child link="LW2_1"/>
-  <axis xyz="0.0 -1.0 0.0"/>
+  <axis xyz="0.0 1.0 0.0"/>
 </joint>
 <joint name="LW1" type="continuous">
@@ -193,5 +193,5 @@
   <child link="Holder_1"/>
 </joint>
-<joint name="Rigid 11" type="fixed">
+<joint name="laser" type="fixed">
   <origin xyz="0.235 0.0 0.135" rpy="0 0 0"/>
   <parent link="base_link"/>
