Commit message: Updated with harmonic sdf and gps driver

File: rusty_description/urdf/materials.xacro (robot description, xacro)
@@ -1,5 +1,5 @@
 <?xml version="1.0" ?>
 <robot name="rusty" xmlns:xacro="http://www.ros.org/wiki/xacro" >
-<material name="silver">
+  <material name="silver">
     <color rgba="0.700 0.700 0.700 1.000"/>
   </material>

File: rusty_description/urdf/rusty.xacro (robot description, xacro)
@@ -1,7 +1,7 @@
 <?xml version="1.0" ?>
 <robot name="rusty" xmlns:xacro="http://www.ros.org/wiki/xacro">
-<xacro:include filename="$(find rusty_description)/urdf/materials.xacro" />
-<xacro:include filename="$(find rusty_description)/urdf/rusty.trans" />
-<xacro:include filename="$(find rusty_description)/urdf/rusty.gazebo" />
+<xacro:include filename="/home/siddarth/ros2ws/src/Rusty/rusty_description/urdf/materials.xacro" />
+<!-- <xacro:include filename="/home/siddarth/ros2ws/src/Rusty/rusty_description/urdf/rusty.trans" /> -->
+<!-- <xacro:include filename="/home/siddarth/ros2ws/src/Rusty/rusty_description/urdf/rusty.gazebo" /> -->
 <link name="base_link">
   <inertial>
@@ -13,5 +13,5 @@
     <origin xyz="0 0 0" rpy="0 0 0"/>
     <geometry>
-      <mesh filename="file://$(find rusty_description)/meshes/base_link.stl" scale="0.001 0.001 0.001"/>
+      <mesh filename="file:///home/siddarth/ros2ws/src/Rusty/rusty_description/meshes/base_link.stl" scale="0.001 0.001 0.001"/>
     </geometry>
     <material name="silver"/>
@@ -20,5 +20,5 @@
     <origin xyz="0 0 0" rpy="0 0 0"/>
     <geometry>
-      <mesh filename="file://$(find rusty_description)/meshes/base_link.stl" scale="0.001 0.001 0.001"/>
+      <mesh filename="file:///home/siddarth/ros2ws/src/Rusty/rusty_description/meshes/base_link.stl" scale="0.001 0.001 0.001"/>
     </geometry>
   </collision>
@@ -33,5 +33,5 @@
     <origin xyz="0.095 0.16 -0.05" rpy="0 0 0"/>
     <geometry>
-      <mesh filename="file://$(find rusty_description)/meshes/RW2_1.stl" scale="0.001 0.001 0.001"/>
+      <mesh filename="file:///home/siddarth/ros2ws/src/Rusty/rusty_description/meshes/RW2_1.stl" scale="0.001 0.001 0.001"/>
     </geometry>
     <material name="black"/>
@@ -40,5 +40,5 @@
     <origin xyz="0.095 0.16 -0.05" rpy="0 0 0"/>
     <geometry>
-      <mesh filename="file://$(find rusty_description)/meshes/RW2_1.stl" scale="0.001 0.001 0.001"/>
+      <mesh filename="file:///home/siddarth/ros2ws/src/Rusty/rusty_description/meshes/RW2_1.stl" scale="0.001 0.001 0.001"/>
     </geometry>
   </collision>
@@ -53,5 +53,5 @@
     <origin xyz="-0.095 0.16 -0.05" rpy="0 0 0"/>
     <geometry>
-      <mesh filename="file://$(find rusty_description)/meshes/RW1_1.stl" scale="0.001 0.001 0.001"/>
+      <mesh filename="file:///home/siddarth/ros2ws/src/Rusty/rusty_description/meshes/RW1_1.stl" scale="0.001 0.001 0.001"/>
     </geometry>
     <material name="black"/>
@@ -60,5 +60,5 @@
     <origin xyz="-0.095 0.16 -0.05" rpy="0 0 0"/>
     <geometry>
-      <mesh filename="file://$(find rusty_description)/meshes/RW1_1.stl" scale="0.001 0.001 0.001"/>
+      <mesh filename="file:///home/siddarth/ros2ws/src/Rusty/rusty_description/meshes/RW1_1.stl" scale="0.001 0.001 0.001"/>
     </geometry>
   </collision>
@@ -73,5 +73,5 @@
     <origin xyz="0.095 -0.16 -0.05" rpy="0 0 0"/>
     <geometry>
-      <mesh filename="file://$(find rusty_description)/meshes/LW2_1.stl" scale="0.001 0.001 0.001"/>
+      <mesh filename="file:///home/siddarth/ros2ws/src/Rusty/rusty_description/meshes/LW2_1.stl" scale="0.001 0.001 0.001"/>
     </geometry>
     <material name="black"/>
@@ -80,5 +80,5 @@
     <origin xyz="0.095 -0.16 -0.05" rpy="0 0 0"/>
     <geometry>
-      <mesh filename="file://$(find rusty_description)/meshes/LW2_1.stl" scale="0.001 0.001 0.001"/>
+      <mesh filename="file:///home/siddarth/ros2ws/src/Rusty/rusty_description/meshes/LW2_1.stl" scale="0.001 0.001 0.001"/>
     </geometry>
   </collision>
@@ -93,5 +93,5 @@
     <origin xyz="-0.095 -0.16 -0.05" rpy="0 0 0"/>
     <geometry>
-      <mesh filename="file://$(find rusty_description)/meshes/LW1_1.stl" scale="0.001 0.001 0.001"/>
+      <mesh filename="file:///home/siddarth/ros2ws/src/Rusty/rusty_description/meshes/LW1_1.stl" scale="0.001 0.001 0.001"/>
     </geometry>
     <material name="black"/>
@@ -100,5 +100,5 @@
     <origin xyz="-0.095 -0.16 -0.05" rpy="0 0 0"/>
     <geometry>
-      <mesh filename="file://$(find rusty_description)/meshes/LW1_1.stl" scale="0.001 0.001 0.001"/>
+      <mesh filename="file:///home/siddarth/ros2ws/src/Rusty/rusty_description/meshes/LW1_1.stl" scale="0.001 0.001 0.001"/>
     </geometry>
   </collision>
@@ -113,5 +113,5 @@
     <origin xyz="-0.0 -0.0 -0.15" rpy="0 0 0"/>
     <geometry>
-      <mesh filename="file://$(find rusty_description)/meshes/Holder_1.stl" scale="0.001 0.001 0.001"/>
+      <mesh filename="file:///home/siddarth/ros2ws/src/Rusty/rusty_description/meshes/Holder_1.stl" scale="0.001 0.001 0.001"/>
     </geometry>
     <material name="blue"/>
@@ -120,5 +120,5 @@
     <origin xyz="-0.0 -0.0 -0.15" rpy="0 0 0"/>
     <geometry>
-      <mesh filename="file://$(find rusty_description)/meshes/Holder_1.stl" scale="0.001 0.001 0.001"/>
+      <mesh filename="file:///home/siddarth/ros2ws/src/Rusty/rusty_description/meshes/Holder_1.stl" scale="0.001 0.001 0.001"/>
     </geometry>
   </collision>
@@ -133,5 +133,5 @@
     <origin xyz="-0.235 -0.0 -0.135" rpy="0 0 0"/>
     <geometry>
-      <mesh filename="file://$(find rusty_description)/meshes/Lidar_1.stl" scale="0.001 0.001 0.001"/>
+      <mesh filename="file:///home/siddarth/ros2ws/src/Rusty/rusty_description/meshes/Lidar_1.stl" scale="0.001 0.001 0.001"/>
     </geometry>
     <material name="orange"/>
@@ -140,5 +140,5 @@
     <origin xyz="-0.235 -0.0 -0.135" rpy="0 0 0"/>
     <geometry>
-      <mesh filename="file://$(find rusty_description)/meshes/Lidar_1.stl" scale="0.001 0.001 0.001"/>
+      <mesh filename="file:///home/siddarth/ros2ws/src/Rusty/rusty_description/meshes/Lidar_1.stl" scale="0.001 0.001 0.001"/>
     </geometry>
   </collision>
@@ -153,5 +153,5 @@
     <origin xyz="-0.222588 -0.012099 -0.15" rpy="0 0 0"/>
     <geometry>
-      <mesh filename="file://$(find rusty_description)/meshes/Camera_1.stl" scale="0.001 0.001 0.001"/>
+      <mesh filename="file:///home/siddarth/ros2ws/src/Rusty/rusty_description/meshes/Camera_1.stl" scale="0.001 0.001 0.001"/>
     </geometry>
     <material name="red"/>
@@ -160,5 +160,5 @@
     <origin xyz="-0.222588 -0.012099 -0.15" rpy="0 0 0"/>
     <geometry>
-      <mesh filename="file://$(find rusty_description)/meshes/Camera_1.stl" scale="0.001 0.001 0.001"/>
+      <mesh filename="file:///home/siddarth/ros2ws/src/Rusty/rusty_description/meshes/Camera_1.stl" scale="0.001 0.001 0.001"/>
     </geometry>
   </collision>
@@ -168,5 +168,5 @@
   <parent link="base_link"/>
   <child link="RW2_1"/>
-  <axis xyz="0.0 1.0 0.0"/>
+  <axis xyz="0.0 0.0 1.0"/>
 </joint>
 <joint name="RW1" type="continuous">
@@ -174,5 +174,5 @@
   <parent link="base_link"/>
   <child link="RW1_1"/>
-  <axis xyz="0.0 1.0 0.0"/>
+  <axis xyz="0.0 0.0 1.0"/>
 </joint>
 <joint name="LW2" type="continuous">
@@ -180,5 +180,5 @@
   <parent link="base_link"/>
   <child link="LW2_1"/>
-  <axis xyz="0.0 1.0 0.0"/>
+  <axis xyz="0.0 0.0 1.0"/>
 </joint>
 <joint name="LW1" type="continuous">
@@ -186,5 +186,5 @@
   <parent link="base_link"/>
   <child link="LW1_1"/>
-  <axis xyz="0.0 1.0 0.0"/>
+  <axis xyz="0.0 0.0 1.0"/>
 </joint>
 <joint name="Rigid 10" type="fixed">
