Commit message: Update rusty.xacro

File: rusty_description/urdf/rusty.xacro (robot description, xacro)
@@ -4,5 +4,5 @@
 <xacro:include filename="$(find rusty_description)/urdf/rusty.trans" />
 <xacro:include filename="$(find rusty_description)/urdf/rusty.gazebo" />
-<link name="base_link">
+<link name="rusty_base">
   <inertial>
     <origin rpy="0 0 0" xyz="0.0002544970294304579 -2.7411733823236023e-17 0.08341254857000653"/>
@@ -166,5 +166,5 @@
 <joint name="RW2" type="continuous">
   <origin rpy="0 0 0" xyz="-0.095 -0.16 0.05"/>
-  <parent link="base_link"/>
+  <parent link="rusty_base"/>
   <child link="RW2_1"/>
   <axis xyz="0.0 1.0 0.0"/>
@@ -172,5 +172,5 @@
 <joint name="RW1" type="continuous">
   <origin rpy="0 0 0" xyz="0.095 -0.16 0.05"/>
-  <parent link="base_link"/>
+  <parent link="rusty_base"/>
   <child link="RW1_1"/>
   <axis xyz="0.0 1.0 0.0"/>
@@ -178,5 +178,5 @@
 <joint name="LW2" type="continuous">
   <origin rpy="0 0 0" xyz="-0.095 0.16 0.05"/>
-  <parent link="base_link"/>
+  <parent link="rusty_base"/>
   <child link="LW2_1"/>
   <axis xyz="0.0 1.0 0.0"/>
@@ -184,5 +184,5 @@
 <joint name="LW1" type="continuous">
   <origin rpy="0 0 0" xyz="0.095 0.16 0.05"/>
-  <parent link="base_link"/>
+  <parent link="rusty_base"/>
   <child link="LW1_1"/>
   <axis xyz="0.0 1.0 0.0"/>
@@ -190,15 +190,15 @@
 <joint name="Rigid10" type="fixed">
   <origin rpy="0 0 0" xyz="0.0 0.0 0.15"/>
-  <parent link="base_link"/>
+  <parent link="rusty_base"/>
   <child link="Holder_1"/>
 </joint>
 <joint name="Rigid11" type="fixed">
   <origin rpy="0 0 0" xyz="0.235 0.0 0.135"/>
-  <parent link="base_link"/>
+  <parent link="rusty_base"/>
   <child link="Lidar_1"/>
 </joint>
 <joint name="Rigid12" type="fixed">
   <origin rpy="0 0 0" xyz="0.222588 0.012099 0.15"/>
-  <parent link="base_link"/>
+  <parent link="rusty_base"/>
   <child link="Camera_1"/>
 </joint>

Commit message: Adding rusty package

File: rusty_description/urdf/rusty.xacro (robot description, xacro)
@@ -35,5 +35,5 @@
       <mesh filename="file://$(find rusty_description)/meshes/RW2_1.stl" scale="0.001 0.001 0.001"/>
     </geometry>
-    <material name="silver"/>
+    <material name="black"/>
   </visual>
   <collision>
@@ -55,5 +55,5 @@
       <mesh filename="file://$(find rusty_description)/meshes/RW1_1.stl" scale="0.001 0.001 0.001"/>
     </geometry>
-    <material name="silver"/>
+    <material name="black"/>
   </visual>
   <collision>
@@ -75,5 +75,5 @@
       <mesh filename="file://$(find rusty_description)/meshes/LW2_1.stl" scale="0.001 0.001 0.001"/>
     </geometry>
-    <material name="silver"/>
+    <material name="black"/>
   </visual>
   <collision>
@@ -95,5 +95,5 @@
       <mesh filename="file://$(find rusty_description)/meshes/LW1_1.stl" scale="0.001 0.001 0.001"/>
     </geometry>
-    <material name="silver"/>
+    <material name="black"/>
   </visual>
   <collision>
@@ -115,5 +115,5 @@
       <mesh filename="file://$(find rusty_description)/meshes/Holder_1.stl" scale="0.001 0.001 0.001"/>
     </geometry>
-    <material name="silver"/>
+    <material name="blue"/>
   </visual>
   <collision>
@@ -135,5 +135,5 @@
       <mesh filename="file://$(find rusty_description)/meshes/Lidar_1.stl" scale="0.001 0.001 0.001"/>
     </geometry>
-    <material name="silver"/>
+    <material name="orange"/>
   </visual>
   <collision>
@@ -155,5 +155,5 @@
       <mesh filename="file://$(find rusty_description)/meshes/Camera_1.stl" scale="0.001 0.001 0.001"/>
     </geometry>
-    <material name="silver"/>
+    <material name="red"/>
   </visual>
   <collision>
@@ -194,5 +194,5 @@
 </joint>
 <joint name="laser" type="fixed">
-  <origin xyz="0.235 0.0 0.135" rpy="0 0 0"/>
+  <origin xyz="0.235 0.0 0.138" rpy="0 0 0"/>
   <parent link="base_link"/>
   <child link="Lidar_1"/>

Commit message: gazebo-classic update

File: rusty_description/urdf/rusty.xacro (robot description, xacro)
@@ -1,7 +1,7 @@
 <?xml version="1.0" ?>
 <robot name="rusty" xmlns:xacro="http://www.ros.org/wiki/xacro">
-<xacro:include filename="/home/siddarth/ros2ws/src/Rusty/rusty_description/urdf/materials.xacro" />
-<!-- <xacro:include filename="/home/siddarth/ros2ws/src/Rusty/rusty_description/urdf/rusty.trans" /> -->
-<!-- <xacro:include filename="/home/siddarth/ros2ws/src/Rusty/rusty_description/urdf/rusty.gazebo" /> -->
+<xacro:include filename="$(find rusty_description)/urdf/materials.xacro" />
+<xacro:include filename="$(find rusty_description)/urdf/rusty.trans" />
+<xacro:include filename="$(find rusty_description)/urdf/rusty.gazebo" />
 <link name="base_link">
   <inertial>
@@ -13,5 +13,5 @@
     <origin xyz="0 0 0" rpy="0 0 0"/>
     <geometry>
-      <mesh filename="file:///home/siddarth/ros2ws/src/Rusty/rusty_description/meshes/base_link.stl" scale="0.001 0.001 0.001"/>
+      <mesh filename="file://$(find rusty_description)/meshes/base_link.stl" scale="0.001 0.001 0.001"/>
     </geometry>
     <material name="silver"/>
@@ -20,5 +20,5 @@
     <origin xyz="0 0 0" rpy="0 0 0"/>
     <geometry>
-      <mesh filename="file:///home/siddarth/ros2ws/src/Rusty/rusty_description/meshes/base_link.stl" scale="0.001 0.001 0.001"/>
+      <mesh filename="file://$(find rusty_description)/meshes/base_link.stl" scale="0.001 0.001 0.001"/>
     </geometry>
   </collision>
@@ -33,12 +33,12 @@
     <origin xyz="0.095 0.16 -0.05" rpy="0 0 0"/>
     <geometry>
-      <mesh filename="file:///home/siddarth/ros2ws/src/Rusty/rusty_description/meshes/RW2_1.stl" scale="0.001 0.001 0.001"/>
-    </geometry>
-    <material name="black"/>
+      <mesh filename="file://$(find rusty_description)/meshes/RW2_1.stl" scale="0.001 0.001 0.001"/>
+    </geometry>
+    <material name="silver"/>
   </visual>
   <collision>
     <origin xyz="0.095 0.16 -0.05" rpy="0 0 0"/>
     <geometry>
-      <mesh filename="file:///home/siddarth/ros2ws/src/Rusty/rusty_description/meshes/RW2_1.stl" scale="0.001 0.001 0.001"/>
+      <mesh filename="file://$(find rusty_description)/meshes/RW2_1.stl" scale="0.001 0.001 0.001"/>
     </geometry>
   </collision>
@@ -53,12 +53,12 @@
     <origin xyz="-0.095 0.16 -0.05" rpy="0 0 0"/>
     <geometry>
-      <mesh filename="file:///home/siddarth/ros2ws/src/Rusty/rusty_description/meshes/RW1_1.stl" scale="0.001 0.001 0.001"/>
-    </geometry>
-    <material name="black"/>
+      <mesh filename="file://$(find rusty_description)/meshes/RW1_1.stl" scale="0.001 0.001 0.001"/>
+    </geometry>
+    <material name="silver"/>
   </visual>
   <collision>
     <origin xyz="-0.095 0.16 -0.05" rpy="0 0 0"/>
     <geometry>
-      <mesh filename="file:///home/siddarth/ros2ws/src/Rusty/rusty_description/meshes/RW1_1.stl" scale="0.001 0.001 0.001"/>
+      <mesh filename="file://$(find rusty_description)/meshes/RW1_1.stl" scale="0.001 0.001 0.001"/>
     </geometry>
   </collision>
@@ -73,12 +73,12 @@
     <origin xyz="0.095 -0.16 -0.05" rpy="0 0 0"/>
     <geometry>
-      <mesh filename="file:///home/siddarth/ros2ws/src/Rusty/rusty_description/meshes/LW2_1.stl" scale="0.001 0.001 0.001"/>
-    </geometry>
-    <material name="black"/>
+      <mesh filename="file://$(find rusty_description)/meshes/LW2_1.stl" scale="0.001 0.001 0.001"/>
+    </geometry>
+    <material name="silver"/>
   </visual>
   <collision>
     <origin xyz="0.095 -0.16 -0.05" rpy="0 0 0"/>
     <geometry>
-      <mesh filename="file:///home/siddarth/ros2ws/src/Rusty/rusty_description/meshes/LW2_1.stl" scale="0.001 0.001 0.001"/>
+      <mesh filename="file://$(find rusty_description)/meshes/LW2_1.stl" scale="0.001 0.001 0.001"/>
     </geometry>
   </collision>
@@ -93,12 +93,12 @@
     <origin xyz="-0.095 -0.16 -0.05" rpy="0 0 0"/>
     <geometry>
-      <mesh filename="file:///home/siddarth/ros2ws/src/Rusty/rusty_description/meshes/LW1_1.stl" scale="0.001 0.001 0.001"/>
-    </geometry>
-    <material name="black"/>
+      <mesh filename="file://$(find rusty_description)/meshes/LW1_1.stl" scale="0.001 0.001 0.001"/>
+    </geometry>
+    <material name="silver"/>
   </visual>
   <collision>
     <origin xyz="-0.095 -0.16 -0.05" rpy="0 0 0"/>
     <geometry>
-      <mesh filename="file:///home/siddarth/ros2ws/src/Rusty/rusty_description/meshes/LW1_1.stl" scale="0.001 0.001 0.001"/>
+      <mesh filename="file://$(find rusty_description)/meshes/LW1_1.stl" scale="0.001 0.001 0.001"/>
     </geometry>
   </collision>
@@ -113,12 +113,12 @@
     <origin xyz="-0.0 -0.0 -0.15" rpy="0 0 0"/>
     <geometry>
-      <mesh filename="file:///home/siddarth/ros2ws/src/Rusty/rusty_description/meshes/Holder_1.stl" scale="0.001 0.001 0.001"/>
-    </geometry>
-    <material name="blue"/>
+      <mesh filename="file://$(find rusty_description)/meshes/Holder_1.stl" scale="0.001 0.001 0.001"/>
+    </geometry>
+    <material name="silver"/>
   </visual>
   <collision>
     <origin xyz="-0.0 -0.0 -0.15" rpy="0 0 0"/>
     <geometry>
-      <mesh filename="file:///home/siddarth/ros2ws/src/Rusty/rusty_description/meshes/Holder_1.stl" scale="0.001 0.001 0.001"/>
+      <mesh filename="file://$(find rusty_description)/meshes/Holder_1.stl" scale="0.001 0.001 0.001"/>
     </geometry>
   </collision>
@@ -133,12 +133,12 @@
     <origin xyz="-0.235 -0.0 -0.135" rpy="0 0 0"/>
     <geometry>
-      <mesh filename="file:///home/siddarth/ros2ws/src/Rusty/rusty_description/meshes/Lidar_1.stl" scale="0.001 0.001 0.001"/>
-    </geometry>
-    <material name="orange"/>
+      <mesh filename="file://$(find rusty_description)/meshes/Lidar_1.stl" scale="0.001 0.001 0.001"/>
+    </geometry>
+    <material name="silver"/>
   </visual>
   <collision>
     <origin xyz="-0.235 -0.0 -0.135" rpy="0 0 0"/>
     <geometry>
-      <mesh filename="file:///home/siddarth/ros2ws/src/Rusty/rusty_description/meshes/Lidar_1.stl" scale="0.001 0.001 0.001"/>
+      <mesh filename="file://$(find rusty_description)/meshes/Lidar_1.stl" scale="0.001 0.001 0.001"/>
     </geometry>
   </collision>
@@ -153,12 +153,12 @@
     <origin xyz="-0.222588 -0.012099 -0.15" rpy="0 0 0"/>
     <geometry>
-      <mesh filename="file:///home/siddarth/ros2ws/src/Rusty/rusty_description/meshes/Camera_1.stl" scale="0.001 0.001 0.001"/>
-    </geometry>
-    <material name="red"/>
+      <mesh filename="file://$(find rusty_description)/meshes/Camera_1.stl" scale="0.001 0.001 0.001"/>
+    </geometry>
+    <material name="silver"/>
   </visual>
   <collision>
     <origin xyz="-0.222588 -0.012099 -0.15" rpy="0 0 0"/>
     <geometry>
-      <mesh filename="file:///home/siddarth/ros2ws/src/Rusty/rusty_description/meshes/Camera_1.stl" scale="0.001 0.001 0.001"/>
+      <mesh filename="file://$(find rusty_description)/meshes/Camera_1.stl" scale="0.001 0.001 0.001"/>
     </geometry>
   </collision>
@@ -168,5 +168,5 @@
   <parent link="base_link"/>
   <child link="RW2_1"/>
-  <axis xyz="0.0 0.0 1.0"/>
+  <axis xyz="0.0 1.0 0.0"/>
 </joint>
 <joint name="RW1" type="continuous">
@@ -174,5 +174,5 @@
   <parent link="base_link"/>
   <child link="RW1_1"/>
-  <axis xyz="0.0 0.0 1.0"/>
+  <axis xyz="0.0 1.0 0.0"/>
 </joint>
 <joint name="LW2" type="continuous">
@@ -180,5 +180,5 @@
   <parent link="base_link"/>
   <child link="LW2_1"/>
-  <axis xyz="0.0 0.0 1.0"/>
+  <axis xyz="0.0 1.0 0.0"/>
 </joint>
 <joint name="LW1" type="continuous">
@@ -186,5 +186,5 @@
   <parent link="base_link"/>
   <child link="LW1_1"/>
-  <axis xyz="0.0 0.0 1.0"/>
+  <axis xyz="0.0 1.0 0.0"/>
 </joint>
 <joint name="Rigid 10" type="fixed">
@@ -194,5 +194,5 @@
 </joint>
 <joint name="laser" type="fixed">
-  <origin xyz="0.235 0.0 0.138" rpy="0 0 0"/>
+  <origin xyz="0.235 0.0 0.135" rpy="0 0 0"/>
   <parent link="base_link"/>
   <child link="Lidar_1"/>

Commit message: ros2 gazebo port

File: rusty_description/urdf/rusty.xacro (robot description, xacro)
@@ -198,5 +198,5 @@
   <child link="Lidar_1"/>
 </joint>
-<joint name="Rigid 12" type="fixed">
+<joint name="camera" type="fixed">
   <origin xyz="0.222588 0.012099 0.15" rpy="0 0 0"/>
   <parent link="base_link"/>
